File: pcb_schematics/SPI_LED_chain.kicad_sch (KiCad schematic)
At the start: 55 parts

Commit message: more schematics
Connections:
- net SOFT_SPI_MISO renamed SOFT_SPI_MOSI
- no-connect marks 0 -> 2
Changed lines of the file:
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@@
 		(color 255 0 0 1)
 	)
+	(no_connect
+		(at 110.49 176.53)
+	)
+	(no_connect
+		(at 110.49 179.07)
+	)
 	(wire
 		(pts
@@
 		)
 	)
-	(global_label "SOFT_SPI_MISO"
+	(global_label "SOFT_SPI_MOSI"
 		(shape input)
 		(at 44.45 38.1 180)
