File: pcb_schematics/pcb_schematics.kicad_pcb (KiCad board)
At the start: 2 copper layers, 27.4 x 23.6 mm, 5 parts, among them U2 SS49E

Commit message: harmora layout design
Other:
- board size 27.4 x 23.6 mm -> 355.8 x 282 mm
- board text added: "->"
- board text added: "1"
- board text added: "11"
- board text added: "13"
- board text added: "2"
- board text added: "3"
- board text added: "4"
- board text added: "6"
- board text added: "7"
- board text added: "9"
- board text added: "<-"
- board text added: "Aeol"
- board text added: "BASS"
- board text added: "CHORD"
- board text added: "CONTROL"
- board text added: "EFFECTS"
- board text added: "EXTENDER"
- board text added: "HARMORA"
- board text added: "I"
- board text added: "II"
- board text added: "III"
- board text added: "INSTRUMENT"
- board text added: "IV"
- board text added: "KEY"
- board text added: "LOOPER"
- board text added: "Locr"
- board text added: "MODE SELECT"
- board text added: "MODIFIER"
- board text added: "OCTAVE"
- board text added: "PATTERN"
- board text added: "PIANO"
- board text added: "STREACHER"
- board text added: "SYNTH"
- board text added: "V"
- board text added: "VI"
- board text added: "VII"
- board text added: "VOLUME"
- board text added: "aug"
- board text added: "b7"
- board text added: "bII"
- board text added: "bIII"
- board text added: "bV"
- board text added: "bVI"
- board text added: "bVII"
- board text added: "dim"
- board text added: "dor"
- board text added: "ion"
- board text added: "lyd"
- board text added: "maj"
- board text added: "min"
- board text added: "mixo"
- board text added: "phry"
- board text added: "sus2"
- board text added: "sus4"
- board text added: "|"

Commit message: schemating...
Other:
- board text added: "HARMORA 328"

Commit message: more schematics
Other:
- board text added: "5"
