File: pcb_schematics/pcb_schematics.kicad_sch (KiCad schematic)
At the start: 4 parts, among them U2 SS49E

Commit message: maximes
Parts:
- removed C1: 100nF, Harmora_PCB_lib:0603_C, symbol Symbols:Capacitor
- removed D1: APA102, Harmora_PCB_lib:APA102 LED, symbol Symbols:APA102 LED
- removed R1: ~, Harmora_PCB_lib:0603_R, symbol Symbols:Resistor
- removed U2: SS49E, Harmora_PCB_lib:SLSS49E-3 Hall Sensor (SOT-23-3), symbol Symbols:SS49E Hall Sensor
Other:
- added sheet Piano (piano_subsheet.kicad_sch)

Commit message: schemating...
Other:
- sheet Piano renamed SPI LED chain
- added sheet Hall Sensors (hall_sensors.kicad_sch)
- sheet SPI LED chain: file piano_subsheet.kicad_sch -> SPI_LED_chain.kicad_sch
Changed lines of the file:
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@@
 	(paper "A4")
 	(sheet
-		(at 121.92 34.29)
+		(at 71.12 17.78)
+		(size 51.435 39.37)
+		(exclude_from_sim no)
+		(in_bom yes)
+		(on_board yes)
+		(dnp no)
+		(fields_autoplaced yes)
+		(stroke
+			(width 0.1524)
+			(type solid)
+		)
+		(fill
+			(color 0 0 0 0.0000)
+		)
+		(property "Sheetname" "Hall Sensors"
+			(at 71.12 17.0684 0)
+			(effects
+				(font
+					(size 1.27 1.27)
+				)
+				(justify left bottom)
+			)
+		)
+		(property "Sheetfile" "hall_sensors.kicad_sch"
+			(at 71.12 57.7346 0)
+			(effects
+				(font
+					(size 1.27 1.27)
+				)
+				(justify left top)
+			)
+		)
+		(instances
+			(project "pcb_schematics"
+				(path "/de43e009-b04c-42c1-b131-cdc664039a0d"
+					(page "3")
+				)
+			)
+		)
+	)
+	(sheet
+		(at 17.78 17.78)
 		(size 49.53 39.37)
 		(exclude_from_sim no)
@@
 			(color 0 0 0 0.0000)
 		)
-		(property "Sheetname" "Piano"
-			(at 121.92 33.5784 0)
+		(property "Sheetname" "SPI LED chain"
+			(at 17.78 17.0684 0)
 			(effects
 				(font
@@
 			)
 		)
-		(property "Sheetfile" "piano_subsheet.kicad_sch"
-			(at 121.92 74.2446 0)
+		(property "Sheetfile" "SPI_LED_chain.kicad_sch"
+			(at 17.78 57.7346 0)
 			(effects
 				(font

Commit message: more schematics
Other:
- sheet Hall Sensors renamed Piano MUX
- added sheet Encoders MUX (encoders_mux.kicad_sch)
- added sheet Expanders (expanders.kicad_sch)
- sheet Piano MUX: file hall_sensors.kicad_sch -> piano_poteniometers_mux.kicad_sch
Changed lines of the file:
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@@
 	(paper "A4")
+	(sheet
+		(at 126.365 17.78)
+		(size 51.435 39.37)
+		(exclude_from_sim no)
+		(in_bom yes)
+		(on_board yes)
+		(dnp no)
+		(fields_autoplaced yes)
+		(stroke
+			(width 0.1524)
+			(type solid)
+		)
+		(fill
+			(color 0 0 0 0.0000)
+		)
+		(property "Sheetname" "Encoders MUX"
+			(at 126.365 17.0684 0)
+			(effects
+				(font
+					(size 1.27 1.27)
+				)
+				(justify left bottom)
+			)
+		)
+		(property "Sheetfile" "encoders_mux.kicad_sch"
+			(at 126.365 57.7346 0)
+			(effects
+				(font
+					(size 1.27 1.27)
+				)
+				(justify left top)
+			)
+		)
+		(instances
+			(project "pcb_schematics"
+				(path "/de43e009-b04c-42c1-b131-cdc664039a0d"
+					(page "4")
+				)
+			)
+		)
+	)
 	(sheet
 		(at 71.12 17.78)
@@
 			(color 0 0 0 0.0000)
 		)
-		(property "Sheetname" "Hall Sensors"
+		(property "Sheetname" "Piano MUX"
 			(at 71.12 17.0684 0)
 			(effects
@@
 			)
 		)
-		(property "Sheetfile" "hall_sensors.kicad_sch"
+		(property "Sheetfile" "piano_poteniometers_mux.kicad_sch"
 			(at 71.12 57.7346 0)
 			(effects
@@
 				)
 			)
+		)
+	)
+	(sheet
+		(at 180.975 17.78)
+		(size 52.07 39.37)
+		(exclude_from_sim no)
+		(in_bom yes)
+		(on_board yes)
+		(dnp no)
+		(fields_autoplaced yes)
+		(stroke
+			(width 0.1524)
+			(type solid)
+		)
+		(fill
+			(color 0 0 0 0.0000)
+		)
+		(property "Sheetname" "Expanders"
+			(at 180.975 17.0684 0)
+			(effects
+				(font
+					(size 1.27 1.27)
+				)
+				(justify left bottom)
+			)
+		)
+		(property "Sheetfile" "expanders.kicad_sch"
+			(at 180.975 57.7346 0)
+			(effects
+				(font
+					(size 1.27 1.27)
+				)
+				(justify left top)
+			)
+		)
+		(instances
+			(project "pcb_schematics"
+				(path "/de43e009-b04c-42c1-b131-cdc664039a0d"
+					(page "5")
+				)
+			)
