File: PCB/MCU_328p.kicad_sch (KiCad schematic)
At the start: 9 parts, among them U14 ATmega328p-AU

Commit message: display, crystal, 32u4<->328p
Parts:
- added C47, C48: 22pF, symbol Symbols:Capacitor 0603
- added C49: 12pF, symbol Symbols:Capacitor 0603
- added U17: 128x64 2.42 inc, symbol Symbols:SPI_OLED_Display
- added Y1: 16Mhz, symbol Symbols:16Mhz_Crystal
Connections:
- net GND: now also U14.3 (GND), C47.2, C48.2, U17.1 (GND), Y1.2, Y1.4
- net VCC: now also C45.2, C46.2, U14.18 (AVCC), U14.4 (VCC), C49.1, U17.2 (VCC)
- net DISPLAY_SS: now reaches U14.13 ((PCINT1/OC1A)PB1)
- net DISPLAY_SS: now also U17.6 (SS)
- net SPI_MOSI: now reaches U14.15 ((PCINT3/OC2A/MOSI)PB3)
- net SPI_MOSI: now also U17.5 (MOSI)
- net SPI_MISO: now reaches U14.16 ((PCINT4/MISO)PB4)
- net SPI_MISO: now also U17.4 (MISO)
- net SPI_SCK: now reaches U14.17 ((SCK/PCINT5)PB5)
- net SPI_SCK: now also U17.3 (SCK)
- net 32U4_SS: now reaches U14.19 (ADC6)
- net at U14.20 (AREF): now also C49.2
- net DMUX_OUT: now reaches U14.31 ((TXD/PCINT17)PD1)
- net 32U4_INT: now reaches U14.32 ((INT0/PCINT18)PD2)
- net XTAL1: now reaches U14.7 ((PCINT6/XTAL1/TOSC1)PB6)
- net XTAL1: now also C47.1, Y1.1
- net XTAL2: now reaches U14.8 ((PCINT7/XTAL2/TOSC2)PB7)
- net XTAL2: now also C48.1, Y1.3
- no-connect marks 0 -> 3
Other:
- added sheet ATmega32u4 (MCU_32u4.kicad_sch)
- note added: "Crystal"
- note added: "VCC Stabilizer"
- moved on the sheet: C44, C45, C46, R10, R11, R12, R13, R9, U14
