File: PCB/Harmora.kicad_pcb (KiCad board)
At the start: 2 copper layers, 355.8 x 282 mm, 5 parts, among them U2 SS49E

Commit message: new schematics
Parts:
- moved C1 150.8 mm to (-79.1, -83.3)
- moved REF** 150.8 mm to (-79.0, -91.5)
- moved REF** 150.8 mm to (-79.1, -95.2)
- moved REF** 150.8 mm to (-79.0, -86.5)
- moved U2 150.8 mm to (-79.0, -86.5)
Other:
- board size 355.8 x 282 mm -> 290.6 x 318.1 mm

Commit message: pcbing
Parts:
- added AM1: CD74HC4067M, Footprints:CD74HC4067M Analog Mux (SOIC-24), F.Cu at (63.9, -29.7)
- added B1: ~, Footprints:Mechanical Switch, F.Cu at (17.4, -127.7)
- added B10: ~, Footprints:Mechanical Switch, F.Cu at (32.5, -67.3)
- added B11: ~, Footprints:Mechanical Switch, F.Cu at (47.6, -127.7)
- added B12: ~, Footprints:Mechanical Switch, F.Cu at (47.6, -112.6)
- added B13: ~, Footprints:Mechanical Switch, F.Cu at (47.6, -97.5)
- added B14: ~, Footprints:Mechanical Switch, F.Cu at (47.6, -82.4)
- added B15: ~, Footprints:Mechanical Switch, F.Cu at (47.6, -67.3)
- added B16: ~, Footprints:Mechanical Switch, F.Cu at (62.7, -127.7)
- added B17: ~, Footprints:Mechanical Switch, F.Cu at (62.7, -112.6)
- added B18: ~, Footprints:Mechanical Switch, F.Cu at (62.7, -97.5)
- added B19: ~, Footprints:Mechanical Switch, F.Cu at (62.7, -82.4)
- added B2: ~, Footprints:Mechanical Switch, F.Cu at (17.4, -112.6)
- added B20: ~, Footprints:Mechanical Switch, F.Cu at (62.7, -67.3)
- added B21: ~, Footprints:Mechanical Switch, F.Cu at (77.8, -127.7)
- added B22: ~, Footprints:Mechanical Switch, F.Cu at (77.8, -112.6)
- added B23: ~, Footprints:Mechanical Switch, F.Cu at (77.8, -97.5)
- added B24: ~, Footprints:Mechanical Switch, F.Cu at (77.8, -82.4)
- added B25: ~, Footprints:Mechanical Switch, F.Cu at (77.8, -67.3)
- added B3: ~, Footprints:Mechanical Switch, F.Cu at (17.4, -97.5)
- added B4: ~, Footprints:Mechanical Switch, F.Cu at (17.4, -82.4)
- added B5: ~, Footprints:Mechanical Switch, F.Cu at (17.4, -67.3)
- added B6: ~, Footprints:Mechanical Switch, F.Cu at (32.5, -127.7)
- added B7: ~, Footprints:Mechanical Switch, F.Cu at (32.5, -112.6)
- added B8: ~, Footprints:Mechanical Switch, F.Cu at (32.5, -97.5)
- added B9: ~, Footprints:Mechanical Switch, F.Cu at (32.5, -82.4)
- added C1: 100nF, Footprints:0603_C, F.Cu at (157.2, 162.6)
- added C10: 100nF, Footprints:0603_C, F.Cu at (223.9, 134.0)
- added C11: 100nF, Footprints:0603_C, F.Cu at (243.0, 134.0)
- added C12: 100nF, Footprints:0603_C, F.Cu at (262.0, 134.0)
- added C13: 22uF, Footprints:C_Electrolytic_4x5.4, F.Cu at (126.6, -21.2)
- added C14: 100nF, Footprints:0603_C, F.Cu at (128.9, -27.9)
- added C15: 100nF, Footprints:0603_C, F.Cu at (128.9, -25.4)
- added C16: 100nF, Footprints:0603_C, F.Cu at (132.9, -40.5)
- added C17: 100nF, Footprints:0603_C, F.Cu at (132.9, -38.0)
- added C18: 100nF, Footprints:0603_C, F.Cu at (132.9, -35.4)
- added C19: 100nF, Footprints:0603_C, F.Cu at (132.9, -32.9)
- added C2: 100nF, Footprints:0603_C, F.Cu at (176.2, 162.6)
- added C20: 100nF, Footprints:0603_C, F.Cu at (132.9, -30.4)
- added C21: 100nF, Footprints:0603_C, F.Cu at (132.9, -27.9)
- added C22: 100nF, Footprints:0603_C, F.Cu at (132.9, -25.4)
- added C23: 100nF, Footprints:0603_C, F.Cu at (136.9, -40.5)
- added C24: 100nF, Footprints:0603_C, F.Cu at (136.9, -38.0)
- added C25: 100nF, Footprints:0603_C, F.Cu at (136.9, -35.4)
- added C26: 100nF, Footprints:0603_C, F.Cu at (136.9, -32.9)
- added C27: 100nF, Footprints:0603_C, F.Cu at (136.9, -30.4)
- added C28: 22uF, Footprints:C_Electrolytic_4x5.4, F.Cu at (126.6, -15.3)
- added C29: 22uF, Footprints:C_Electrolytic_4x5.4, F.Cu at (126.6, -9.47)
- added C3: 100nF, Footprints:0603_C, F.Cu at (195.3, 162.6)
- added C30: 100nF, Footprints:0603_C, F.Cu at (154.3, 171.4)
- added C31: 100nF, Footprints:0603_C, F.Cu at (173.3, 171.4)
- added C32: 100nF, Footprints:0603_C, F.Cu at (192.4, 171.4)
- added C33: 100nF, Footprints:0603_C, F.Cu at (211.4, 171.4)
- added C34: 100nF, Footprints:0603_C, F.Cu at (230.5, 171.5)
- added C35: 100nF, Footprints:0603_C, F.Cu at (249.5, 171.4)
- added C36: 100nF, Footprints:0603_C, F.Cu at (268.6, 171.4)
- added C37: 100nF, Footprints:0603_C, F.Cu at (163.8, 142.9)
- added C38: 100nF, Footprints:0603_C, F.Cu at (182.9, 142.9)
- added C39: 100nF, Footprints:0603_C, F.Cu at (221.1, 142.9)
- added C4: 100nF, Footprints:0603_C, F.Cu at (214.3, 162.6)
- added C40: 100nF, Footprints:0603_C, F.Cu at (240.1, 142.9)
- added C41: 100nF, Footprints:0603_C, F.Cu at (259.2, 142.9)
- added C42: 100nF, Footprints:0603_C, F.Cu at (66.5, -58.5)
- added C43: 100nF, Footprints:0603_C, F.Cu at (66.5, -56.0)
- added C45: 100nF, Footprints:0603_C, F.Cu at (130.8, -134.0)
- added C46: 1uF, Footprints:0603_C, F.Cu at (130.8, -131.5)
- added C47: 22pF, Footprints:0603_C, F.Cu at (130.8, -128.9)
- added C48: 22pF, Footprints:0603_C, F.Cu at (130.8, -126.4)
- added C49: 100nF, Footprints:0603_C, F.Cu at (130.8, -123.9)
- added C5: 100nF, Footprints:0603_C, F.Cu at (233.4, 162.6)
- added C50: 100nF, Footprints:0603_C, F.Cu at (130.8, -121.4)
- added C51: 100nF, Footprints:0603_C, F.Cu at (11.9, -19.9)
- added C52: 100nF, Footprints:0603_C, F.Cu at (11.9, -17.3)
- added C53: 100nF, Footprints:0603_C, F.Cu at (11.9, -14.8)
- added C54: 100nF, Footprints:0603_C, F.Cu at (11.9, -12.3)
- added C55: 22pF, Footprints:0603_C, F.Cu at (11.9, -9.81)
- added C56: 22pF, Footprints:0603_C, F.Cu at (11.9, -7.30)
- added C57: 1uF, Footprints:0603_C, F.Cu at (11.9, -4.79)
- added C58: 100nF, Footprints:0603_C, F.Cu at (130.8, -118.9)
- added C59: 1nF, Footprints:0603_C, F.Cu at (15.9, -19.9)
- added C6: 100nF, Footprints:0603_C, F.Cu at (252.4, 162.6)
- added C60: 100nF, Footprints:0603_C, F.Cu at (134.8, -134.0)
- added C61: 100nF, Footprints:0603_C, F.Cu at (15.9, -17.3)
- added C62: 1uF, Footprints:0603_C, F.Cu at (15.9, -14.8)
- added C63: 100nF, Footprints:0603_C, F.Cu at (15.9, -12.3)
- added C64: 100nF, Footprints:0603_C, F.Cu at (134.8, -131.5)
- added C7: 100nF, Footprints:0603_C, F.Cu at (271.5, 162.6)
- added C8: 100nF, Footprints:0603_C, F.Cu at (166.7, 134.0)
- added C9: 100nF, Footprints:0603_C, F.Cu at (185.7, 134.0)
- added D1: APA102, Footprints:APA102 LED, F.Cu at (157.2, 166.4)
- added D10: APA102, Footprints:APA102 LED, F.Cu at (223.9, 137.8)
- added D11: APA102, Footprints:APA102 LED, F.Cu at (243.0, 137.8)
- added D12: APA102, Footprints:APA102 LED, F.Cu at (262.0, 137.8)
- added D13: APA102, Footprints:APA102 LED, F.Cu at (100.7, -4.87)
- added D14: APA102, Footprints:APA102 LED, F.Cu at (100.7, 1.83)
- added D15: APA102, Footprints:APA102 LED, F.Cu at (109.6, -38.4)
- added D16: APA102, Footprints:APA102 LED, F.Cu at (109.6, -31.7)
- added D17: APA102, Footprints:APA102 LED, F.Cu at (109.6, -25.0)
- added D18: APA102, Footprints:APA102 LED, F.Cu at (109.6, -18.3)
- added D19: APA102, Footprints:APA102 LED, F.Cu at (109.6, -11.6)
- added D2: APA102, Footprints:APA102 LED, F.Cu at (176.2, 166.4)
- added D20: APA102, Footprints:APA102 LED, F.Cu at (109.6, -4.87)
- added D21: APA102, Footprints:APA102 LED, F.Cu at (109.6, 1.83)
- added D22: APA102, Footprints:APA102 LED, F.Cu at (118.5, -38.4)
- added D23: APA102, Footprints:APA102 LED, F.Cu at (118.5, -31.7)
- added D24: APA102, Footprints:APA102 LED, F.Cu at (118.5, -25.0)
- added D25: APA102, Footprints:APA102 LED, F.Cu at (118.5, -18.3)
- added D26: APA102, Footprints:APA102 LED, F.Cu at (118.5, -11.6)
- added D27: ~, Footprints:TVS Diode SOD-123FL, F.Cu at (25.0, -5.08)
- added D3: APA102, Footprints:APA102 LED, F.Cu at (195.3, 166.4)
- added D4: APA102, Footprints:APA102 LED, F.Cu at (214.3, 166.4)
- added D5: APA102, Footprints:APA102 LED, F.Cu at (233.4, 166.4)
- added D6: APA102, Footprints:APA102 LED, F.Cu at (252.4, 166.4)
- added D7: APA102, Footprints:APA102 LED, F.Cu at (271.5, 166.4)
- added D8: APA102, Footprints:APA102 LED, F.Cu at (166.7, 137.8)
- added D9: APA102, Footprints:APA102 LED, F.Cu at (185.7, 137.8)
- added DM1: 74LVC1G157, Footprints:74LVC1G157 SOT-363 2_1 MUX, F.Cu at (108.4, -121.3)
- added DM2: 74AC151SC, Footprints:74AC151SC SOIC-16 8_1 MUX, F.Cu at (111.1, -129.3)
- added DM3: 74AC151SC, Footprints:74AC151SC SOIC-16 8_1 MUX, F.Cu at (121.5, -129.3)
- added EN1: ~, Footprints:Rotary Encoder EC11E, F.Cu at (89.3, -130.1)
- added EN2: ~, Footprints:Rotary Encoder EC11E, F.Cu at (89.3, -114.8)
- added EN3: ~, Footprints:Rotary Encoder EC11E, F.Cu at (89.3, -99.6)
- added EN4: ~, Footprints:Rotary Encoder EC11E, F.Cu at (89.3, -84.3)
- added EN5: ~, Footprints:Rotary Encoder EC11E, F.Cu at (89.3, -69.1)
- added EN6: ~, Footprints:Rotary Encoder EC11E, F.Cu at (89.3, -53.8)
- added EX1: ~, Footprints:MCP23017 GPIO Expander, F.Cu at (45.0, -50.0)
- added EX2: ~, Footprints:MCP23017 GPIO Expander, F.Cu at (58.0, -50.0)
- added F1: 500mA, Footprints:Resettable Fuse 1206, F.Cu at (30.8, -5.11)
- added FB1: 600Ω@100MHz, Footprints:0603_FB, F.Cu at (134.8, -128.9)
- added J1: USBC, Footprints:USB C Receptacle USB2.0 16PIN, F.Cu at (33.8, -32.4)
- added J2: ~, Footprints:ISP port, F.Cu at (143.1, -120.8)
- added J3: ~, Footprints:ISP port, F.Cu at (38.5, -12.4)
- added J4: DIN 5, Footprints:DIN_5 port, F.Cu at (18.9, -29.4)
- added R1: 10k, Footprints:0603_R, F.Cu at (67.6, -14.9)
- added R10: 5.1k, Footprints:0603_R, F.Cu at (134.8, -123.9)
- added R11: 330, Footprints:0603_R, F.Cu at (15.9, -9.81)
- added R12: 22, Footprints:0603_R, F.Cu at (134.8, -121.4)
- added R13: 22, Footprints:0603_R, F.Cu at (134.8, -118.9)
- added R14: 22, Footprints:0603_R, F.Cu at (15.9, -7.30)
- added R15: 22, Footprints:0603_R, F.Cu at (15.9, -4.79)
- added R16: 5.1k, Footprints:0603_R, F.Cu at (19.9, -19.9)
- added R17: 5.1k, Footprints:0603_R, F.Cu at (19.9, -17.3)
- added R18: 10k, Footprints:0603_R, F.Cu at (138.8, -134.0)
- added R19: 10k, Footprints:0603_R, F.Cu at (19.9, -14.8)
- added R2: 2.2k, Footprints:0603_R, F.Cu at (67.6, -12.4)
- added R20: 330, Footprints:0603_R, F.Cu at (138.8, -131.5)
- added R21: 10k, Footprints:0603_R, F.Cu at (138.8, -128.9)
- added R22: 2.2k, Footprints:0603_R, F.Cu at (138.8, -126.4)
- added R23: 330, Footprints:0603_R, F.Cu at (19.9, -12.3)
- added R3: 2.2k, Footprints:0603_R, F.Cu at (67.6, -9.87)
- added R4: 2.2k, Footprints:0603_R, F.Cu at (71.6, -19.9)
- added R5: 2.2k, Footprints:0603_R, F.Cu at (71.6, -17.4)
- added R6: 10k, Footprints:0603_R, F.Cu at (71.6, -14.9)
- added R7: 10k, Footprints:0603_R, F.Cu at (71.6, -12.4)
- added R8: 10k, Footprints:0603_R, F.Cu at (71.6, -9.87)
- added R9: 5.1k, Footprints:0603_R, F.Cu at (134.8, -126.4)
- added REF**: Magnetic Switch, Footprints:Magnetic Switch, F.Cu at (262.0, 142.9)
- added REF**: Magnetic Switch, Footprints:Magnetic Switch, F.Cu at (166.7, 142.9)
- added REF**: Magnetic Switch, Footprints:Magnetic Switch, F.Cu at (157.2, 171.4)
- added REF**: Magnetic Switch, Footprints:Magnetic Switch, F.Cu at (243.0, 142.9)
- added REF**: Magnetic Switch, Footprints:Magnetic Switch, F.Cu at (214.3, 171.4)
- added REF**: Magnetic Switch, Footprints:Magnetic Switch, F.Cu at (252.4, 171.4)
- added REF**: Magnetic Switch, Footprints:Magnetic Switch, F.Cu at (176.2, 171.4)
- added REF**: Magnetic Switch, Footprints:Magnetic Switch, F.Cu at (195.3, 171.4)
- added REF**: Magnetic Switch, Footprints:Magnetic Switch, F.Cu at (223.9, 142.9)
- added REF**: Magnetic Switch, Footprints:Magnetic Switch, F.Cu at (271.5, 171.4)
- added REF**: Magnetic Switch, Footprints:Magnetic Switch, F.Cu at (233.4, 171.5)
- added REF**: Magnetic Switch, Footprints:Magnetic Switch, F.Cu at (185.7, 142.9)
- added S1: ~, Footprints:MTS-102 Switch, F.Cu at (15.2, -47.8)
- added S2: ~, Footprints:MTS-102 Switch, F.Cu at (24.7, -47.8)
- added S3: ~, Footprints:MTS-102 Switch, F.Cu at (34.2, -47.8)
- added U1: SS49E, Footprints:SLSS49E-3 Hall Sensor (SOT-23-3), F.Cu at (157.2, 171.4)
- added U10: SS49E, Footprints:SLSS49E-3 Hall Sensor (SOT-23-3), F.Cu at (223.9, 142.9)
- added U11: SS49E, Footprints:SLSS49E-3 Hall Sensor (SOT-23-3), F.Cu at (243.0, 142.9)
- added U12: SS49E, Footprints:SLSS49E-3 Hall Sensor (SOT-23-3), F.Cu at (262.0, 142.9)
- added U14: ATmega328p-AU, Footprints:ATMEGA328P-AU, F.Cu at (134.4, -112.0)
- added U15: ATMEGA32U4-AU, Footprints:ATMEGA32U4-AU, F.Cu at (29.1, -13.9)
- added U16: USBLC6-2SC6, Footprints:ESD Prot SOT-23-6, F.Cu at (37.2, -25.3)
- added U17: 128x64 2.42 inc, Footprints:SPI Screen PinHeader, F.Cu at (147.7, -127.2)
- added U2: SS49E, Footprints:SLSS49E-3 Hall Sensor (SOT-23-3), F.Cu at (176.2, 171.4)
- added U3: SS49E, Footprints:SLSS49E-3 Hall Sensor (SOT-23-3), F.Cu at (195.3, 171.4)
- added U4: SS49E, Footprints:SLSS49E-3 Hall Sensor (SOT-23-3), F.Cu at (214.3, 171.4)
- added U5: SS49E, Footprints:SLSS49E-3 Hall Sensor (SOT-23-3), F.Cu at (233.4, 171.5)
- added U6: SS49E, Footprints:SLSS49E-3 Hall Sensor (SOT-23-3), F.Cu at (252.4, 171.4)
- added U7: SS49E, Footprints:SLSS49E-3 Hall Sensor (SOT-23-3), F.Cu at (271.5, 171.4)
- added U8: SS49E, Footprints:SLSS49E-3 Hall Sensor (SOT-23-3), F.Cu at (166.7, 142.9)
- added U9: SS49E, Footprints:SLSS49E-3 Hall Sensor (SOT-23-3), F.Cu at (185.7, 142.9)
- added Y1: 16Mhz, Footprints:Crystal Oscillator 16MHz, F.Cu at (144.1, -132.3)
- added Y2: 16Mhz, Footprints:Crystal Oscillator 16MHz, F.Cu at (31.3, -24.9)
Routing:
- net Net-(D3-CKO): track 0.00 -> 12.7 mm
- net Net-(D2-SDO): track 0.00 -> 12.7 mm
- net Net-(D2-CKO): track 0.00 -> 12.7 mm
- net Net-(D1-SDO): track 0.00 -> 12.7 mm
- net Net-(D1-CKO): track 0.00 -> 12.7 mm
Other:
- board size 290.6 x 318.1 mm -> 290.6 x 316.5 mm

Commit message: led chain
Parts:
- removed R1, R6, R7, R8: 10k, Footprints:0603_R
- removed the REF** at (262.0, 142.9)
- removed the REF** at (166.7, 142.9)
- removed the REF** at (157.2, 171.4)
- removed the REF** at (243.0, 142.9)
- removed the REF** at (214.3, 171.4)
- removed the REF** at (252.4, 171.4)
- removed the REF** at (176.2, 171.4)
- removed the REF** at (195.3, 171.4)
- removed the REF** at (223.9, 142.9)
- removed the REF** at (271.5, 171.4)
- removed the REF** at (233.4, 171.5)
- removed the REF** at (185.7, 142.9)
- removed U17: 128x64 2.42 inc, Footprints:SPI Screen PinHeader
- added J5: 128x64 2.42 inc, Footprints:SPI Screen PinHeader, B.Cu at (252.4, 81.0)
- added P1: 10k, Footprints:Rotary Potentiometer RK09, B.Cu at (71.4, 81.0)
- added P2: 10k, Footprints:Rotary Potentiometer RK09, B.Cu at (71.4, 109.5)
- added P3: 10k, Footprints:Rotary Potentiometer RK09, B.Cu at (100.0, 81.0)
- added P4: 10k, Footprints:Rotary Potentiometer RK09, B.Cu at (100.0, 109.5)
- added REF**: Magnetic Switch, Footprints:Magnetic Switch, B.Cu at (157.2, 157.2)
- added REF**: Magnetic Switch, Footprints:Magnetic Switch, B.Cu at (90.5, 185.7)
- added REF**: Magnetic Switch, Footprints:Magnetic Switch, B.Cu at (128.6, 185.7)
- added REF**: Magnetic Switch, Footprints:Magnetic Switch, B.Cu at (109.5, 185.7)
- added REF**: Magnetic Switch, Footprints:Magnetic Switch, B.Cu at (100.0, 157.2)
- added REF**: Magnetic Switch, Footprints:Magnetic Switch, B.Cu at (176.2, 157.2)
- added REF**: Magnetic Switch, Footprints:Magnetic Switch, B.Cu at (185.7, 185.7)
- added REF**: Magnetic Switch, Footprints:Magnetic Switch, B.Cu at (166.7, 185.7)
- added REF**: Magnetic Switch, Footprints:Magnetic Switch, B.Cu at (71.4, 185.7)
- added REF**: Magnetic Switch, Footprints:Magnetic Switch, B.Cu at (119.1, 157.2)
- added REF**: Magnetic Switch, Footprints:Magnetic Switch, B.Cu at (81.0, 157.2)
- added REF**: Magnetic Switch, Footprints:Magnetic Switch, B.Cu at (147.6, 185.7)
- B1, B10, B11, B12, B13, B14, B15, B16, B17, B18, B19, B2, B20, B21, B22, B23, B24, B25, B3, B4, B5, B6, B7, B8, B9, EN1, EN2, EN3, EN4, EN5, EN6, S1, S2, S3: moved to B.Cu
- moved B6 428.6 mm to (314.3, 195.3), turned to 180 degrees
- moved B9 409.4 mm to (333.4, 195.3), turned to 180 degrees
- moved B8 406.7 mm to (333.4, 176.2), turned to 180 degrees
- moved B7 404.1 mm to (333.4, 157.2), turned to 180 degrees
- moved B3 403.6 mm to (295.3, 195.3), turned to 180 degrees
- moved B2 400.7 mm to (295.3, 176.2), turned to 180 degrees
- moved B1 397.9 mm to (295.3, 157.2), turned to 180 degrees
- moved B5 384.0 mm to (314.3, 176.2), turned to 180 degrees
- moved B4 381.5 mm to (314.3, 157.2), turned to 180 degrees
- moved B11 379.9 mm to (247.7, 195.3)
- moved B13 365.6 mm to (266.7, 195.3)
- moved B12 362.5 mm to (266.7, 176.2)
- moved S3 340.3 mm to (333.4, 114.3), turned to 180 degrees
- moved B20 336.9 mm to (333.4, 133.3)
- moved S2 331.9 mm to (314.3, 114.2), turned to 180 degrees
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Routing:
- net Net-(D7-SDO): track 0.00 -> 123.7 mm
- net Net-(D7-CKO): track 0.00 -> 122.0 mm
- net Net-(D3-CKO): track 12.7 -> 0.00 mm
- net Net-(D2-SDO): track 12.7 -> 0.00 mm
- net Net-(D2-CKO): track 12.7 -> 0.00 mm
- net Net-(D1-SDO): track 12.7 -> 0.00 mm
- net Net-(D1-CKO): track 12.7 -> 0.00 mm
Other:
- board size 290.6 x 316.5 mm -> 659.3 x 307 mm
- board text removed: "->"
- board text removed: "5"
- board text removed: "<-"
- board text removed: "HARMORA 328"

Commit message: pcb: piano done
Parts:
- moved EX1 265.2 mm to (213.5, 154.7)
- moved R5 261.0 mm to (146.5, 134.5)
- moved EX2 227.3 mm to (218.5, 111.1)
- moved C27 221.6 mm to (333.4, 72.2)
- moved C26 206.2 mm to (314.3, 72.2)
- moved C72 196.0 mm to (49.0, 164.7)
- moved C25 191.5 mm to (295.2, 72.2)
- moved C71 180.1 mm to (43.0, 150.1)
- moved R3 167.1 mm to (146.5, 129.5)
- moved C70 167.1 mm to (109.5, 145.0), turned to 90 degrees
- moved R1 165.0 mm to (146.5, 132.5)
- moved R4 163.6 mm to (146.5, 128.0)
- moved R2 161.5 mm to (146.5, 131.0)
- moved C6 95.3 mm to (71.4, 177.0)
- moved C7 95.3 mm to (90.5, 177.0)
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- renumbered C13 to C70, C29 to C71, C28 to C72, C46 to C73, C57 to C74, C59 to C75, C62 to C76, C55 to C77, C56 to C78, C47 to C79, C48 to C80, D20 to D13, D21 to D14, D22 to D15, D23 to D16, D13 to D17, D14 to D18, D15 to D19, D16 to D20, D17 to D21, D18 to D22, D19 to D23, R2 to R1, R12 to R10, R13 to R11, R14 to R12, R15 to R13, R18 to R14, R19 to R15, R21 to R16, R20 to R17, R23 to R18, R11 to R19, R3 to R2, R4 to R3, R5 to R4, R22 to R5, R9 to R6, R10 to R7, R16 to R8, R17 to R9
Connections:
- C1 pad 1: Net-(U2-VCC) -> GND
- C1 pad 2: Net-(U2-GND) -> VCC
- J5 pad 1: (no net) -> GND
- J5 pad 2: (no net) -> VCC
- J5 pad 3: (no net) -> /SPI_SCK
- J5 pad 4: (no net) -> /DISPLAY_DR
- J5 pad 5: (no net) -> /SPI_MOSI
- J5 pad 6: (no net) -> /DISPLAY_SS
- J5 pad 7: (no net) -> DISPLAY_RST
- R1 pad 1: Net-(AM1-I15) -> Net-(AM1-I11)
- R1 pad 2: Net-(P1-Pad2) -> Net-(P4-Pad2)
- R2 pad 1: Net-(AM1-I14) -> Net-(AM1-I10)
- R2 pad 2: Net-(P2-Pad2) -> Net-(P3-Pad2)
- R3 pad 1: Net-(AM1-I13) -> Net-(AM1-I9)
- R3 pad 2: Net-(P3-Pad2) -> Net-(P1-Pad2)
- R4 pad 1: Net-(AM1-I12) -> Net-(AM1-I8)
- R4 pad 2: Net-(P4-Pad2) -> Net-(P2-Pad2)
- U1 pad 3: Net-(AM1-I0) -> Net-(AM1-I1)
- U10 pad 3: Net-(AM1-I9) -> Net-(AM1-I13)
- U11 pad 3: Net-(AM1-I10) -> Net-(AM1-I12)
- U12 pad 3: Net-(AM1-I11) -> Net-(AM1-I0)
- U2 pad 3: Net-(AM1-I1) -> Net-(AM1-I2)
- U2 pad 1: Net-(U2-VCC) -> VCC
- U2 pad 2: unconnected-(U2-OUTPUT-Pad2) -> GND
- U2 pad 3: Net-(U2-GND) -> Net-(AM1-I2)
- U3 pad 3: Net-(AM1-I2) -> Net-(AM1-I3)
- U4 pad 3: Net-(AM1-I3) -> Net-(AM1-I4)
- U5 pad 3: Net-(AM1-I4) -> Net-(AM1-I5)
- U6 pad 3: Net-(AM1-I5) -> Net-(AM1-I6)
- U7 pad 3: Net-(AM1-I6) -> Net-(AM1-I7)
- U8 pad 3: Net-(AM1-I7) -> Net-(AM1-I15)
- U9 pad 3: Net-(AM1-I8) -> Net-(AM1-I14)
Routing:
- net Net-(D16-CKO): track 0.00 -> 271.3 mm
- net Net-(D16-SDO): track 0.00 -> 270.3 mm
- net Net-(AM1-I7): track 0.00 -> 254.8 mm
- net Net-(AM1-I6): track 0.00 -> 230.8 mm
- net Net-(AM1-I5): track 0.00 -> 211.7 mm
- net Net-(AM1-I0): track 0.00 -> 194.1 mm
- net Net-(AM1-I12): track 0.00 -> 190.1 mm
- net Net-(AM1-I4): track 0.00 -> 189.9 mm
- net Net-(AM1-I3): track 0.00 -> 168.7 mm
- net Net-(AM1-I13): track 0.00 -> 149.4 mm
- net Net-(AM1-I2): track 0.00 -> 147.8 mm
- net Net-(D5-SDO): track 0.00 -> 144.5 mm
- net Net-(D5-CKO): track 0.00 -> 143.9 mm
- net Net-(AM1-I14): track 0.00 -> 127.5 mm
- net Net-(AM1-I1): track 0.00 -> 126.6 mm
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
Commit message: longahh day
Parts:
- moved U15 270.9 mm to (272.0, 106.0)
- moved DM3 255.4 mm to (171.2, 121.2)
- moved DM2 253.0 mm to (142.8, 121.7)
- moved DM1 250.6 mm to (157.0, 124.5), turned to -90 degrees
- moved AM1 66.2 mm to (71.3, 134.0)
- moved R1 66.2 mm to (80.3, 132.5)
- moved R2 66.2 mm to (80.3, 131.0)
- moved R3 66.2 mm to (80.3, 129.5)
- moved R4 66.2 mm to (80.3, 128.0)
- moved R5 66.2 mm to (80.3, 134.5)
- moved EX1 27.6 mm to (195.3, 134.0), turned to -90 degrees
- moved EX2 20.3 mm to (234.5, 98.6)
- moved U14 10.0 mm to (157.0, 135.5)
- moved C70 1.00 mm to (108.5, 145.0)
Connections:
- B24 pad 1: Net-(EX2-GPA6) -> Net-(EX1-GPB7)
- B25 pad 1: Net-(EX2-GPA7) -> Net-(EX1-GPA0)
- B4 pad 1: Net-(EX1-GPB3) -> Net-(EX2-GPA7)
- B7 pad 1: Net-(EX1-GPB6) -> Net-(EX2-GPA6)
- B8 pad 1: Net-(EX1-GPB7) -> Net-(EX1-GPB3)
- B9 pad 1: Net-(EX1-GPA0) -> Net-(EX1-GPB6)
- DM3 pad 12: unconnected-(DM3-I7-Pad12) -> DISPLAY_RST
- DM3 pad 13: DISPLAY_RST -> unconnected-(DM3-I6-Pad13)
Routing:
- net Net-(P2-Pad2): track 81.4 -> 15.0 mm
- net Net-(P1-Pad2): track 108.2 -> 45.7 mm
- net Net-(AM1-I14): track 127.5 -> 65.2 mm
- net Net-(AM1-I15): track 105.7 -> 43.4 mm
- net Net-(AM1-I13): track 149.4 -> 87.1 mm
- net Net-(AM1-I12): track 190.1 -> 128.1 mm
- net Net-(P3-Pad2): track 109.5 -> 50.4 mm
- net Net-(AM1-I1): track 126.6 -> 67.9 mm
- net Net-(AM1-I2): track 147.8 -> 89.7 mm
- net Net-(AM1-I3): track 168.7 -> 111.3 mm
- net Net-(AM1-I7): track 254.8 -> 197.7 mm
- net Net-(AM1-I4): track 189.9 -> 132.8 mm
- net Net-(AM1-I6): track 230.8 -> 173.7 mm
- net Net-(AM1-I5): track 211.7 -> 154.7 mm
- net Net-(AM1-I0): track 194.1 -> 144.2 mm
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
Commit message: pc is being
Parts:
- moved C64 278.5 mm to (168.7, 145.0), turned to 180 degrees
- moved R10 268.0 mm to (94.5, 143.5)
- moved R11 266.8 mm to (90.1, 144.1)
- moved C53 242.8 mm to (223.0, 105.0), turned to 90 degrees
- moved C74 233.9 mm to (225.3, 91.0)
- moved C78 230.7 mm to (215.4, 101.2), turned to -90 degrees
- moved C77 230.2 mm to (211.8, 104.3)
- moved C52 227.4 mm to (215.3, 84.3), turned to -90 degrees
- moved C61 223.0 mm to (205.5, 100.0), turned to 90 degrees
- moved Y2 220.3 mm to (211.9, 101.2)
- moved R15 220.1 mm to (207.6, 100.0), turned to 90 degrees
- moved C51 219.1 mm to (204.7, 84.2), turned to -90 degrees
- moved R12 209.4 mm to (201.5, 89.7)
- moved R8 208.9 mm to (204.5, 78.0), turned to -90 degrees
- moved R13 207.6 mm to (201.5, 88.2)
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Connections:
- B10 pad 1: Net-(EX1-GPA4) -> Net-(EX1-GPA6)
- B11 pad 1: Net-(EX1-GPA5) -> Net-(EX1-GPA4)
- B12 pad 1: Net-(EX1-GPA6) -> Net-(EX1-GPA7)
- B13 pad 1: Net-(EX1-GPA7) -> Net-(EX1-GPA5)
- B14 pad 1: Net-(EX2-GPB0) -> Net-(EX1-GPB7)
- B15 pad 1: Net-(EX2-GPB1) -> Net-(EX1-GPB6)
- B16 pad 1: Net-(EX2-GPB2) -> Net-(EX1-GPB5)
- B17 pad 1: Net-(EX2-GPB3) -> Net-(EX2-GPA0)
- B18 pad 1: Net-(EX2-GPB4) -> Net-(EX2-GPA1)
- B19 pad 1: Net-(EX2-GPB5) -> Net-(EX2-GPA4)
- B2 pad 1: Net-(EX1-GPB1) -> Net-(EX1-GPB3)
- B20 pad 1: Net-(EX2-GPB6) -> Net-(EX2-GPA5)
- B21 pad 1: Net-(EX2-GPA3) -> Net-(EX2-GPB3)
- B22 pad 1: Net-(EX2-GPA4) -> Net-(EX2-GPB2)
- B23 pad 1: Net-(EX2-GPA5) -> Net-(EX2-GPB1)
- B24 pad 1: Net-(EX1-GPB7) -> Net-(EX1-GPA1)
- B3 pad 1: Net-(EX1-GPB2) -> Net-(EX1-GPA3)
- B4 pad 1: Net-(EX2-GPA7) -> Net-(EX2-GPA2)
- B5 pad 1: Net-(EX1-GPB4) -> Net-(EX1-GPB2)
- B6 pad 1: Net-(EX1-GPB5) -> Net-(EX1-GPA2)
- B7 pad 1: Net-(EX2-GPA6) -> Net-(EX2-GPA3)
- B8 pad 1: Net-(EX1-GPB3) -> Net-(EX1-GPB1)
- B9 pad 1: Net-(EX1-GPB6) -> Net-(EX1-GPB4)
- EN4 pad 1: Net-(DM2-I7) -> Net-(DM2-I6)
- EN4 pad 3: Net-(DM2-I6) -> Net-(DM2-I7)
- EN5 pad 1: Net-(DM3-I3) -> Net-(DM3-I2)
- EN5 pad 3: Net-(DM3-I2) -> Net-(DM3-I3)
- EN5 pad 4: Net-(DM3-I5) -> Net-(DM3-I1)
- EN6 pad 1: Net-(DM3-I1) -> Net-(DM3-I4)
- EN6 pad 3: Net-(DM3-I0) -> Net-(DM3-I5)
- EN6 pad 4: Net-(DM3-I4) -> Net-(DM3-I0)
- EX1 pad 22: D_IN_1 -> Net-(EX1-GPA1)
- EX1 pad 23: D_IN_22 -> Net-(EX1-GPA2)
- EX1 pad 24: D_IN_21 -> Net-(EX1-GPA3)
- EX2 pad 5: Net-(EX2-GPB4) -> D_IN_23
- EX2 pad 6: Net-(EX2-GPB5) -> D_IN_22
- EX2 pad 7: Net-(EX2-GPB6) -> D_IN_21
- EX2 pad 8: D_IN_23 -> D_IN_1
- S1 pad 2: Net-(EX2-GPA0) -> Net-(EX2-GPB0)
- S2 pad 2: Net-(EX2-GPA1) -> Net-(EX2-GPA6)
- S3 pad 2: Net-(EX2-GPA2) -> Net-(EX2-GPA7)
- U14 pad 24: /EXP1_INTA -> /EXP1_INTB
- U14 pad 25: /EXP1_INTB -> /EXP1_INTA
Routing:
- net VCC: track 69.6 -> 884.2 mm
- net D_IN_21: track 0.00 -> 194.8 mm
- net D_IN_22: track 0.00 -> 166.9 mm
- net D_IN_1: track 0.00 -> 150.4 mm
- net Net-(EX1-GPB4): track 0.00 -> 143.8 mm
- net D_IN_23: track 0.00 -> 139.2 mm
- net /GPIO Expanders/I2C_SDA: track 0.00 -> 134.3 mm, vias 0 -> 2
- net Net-(EX1-GPB1): track 0.00 -> 125.7 mm
- net /GPIO Expanders/I2C_SCK: track 0.00 -> 124.2 mm
- net Net-(EX1-GPA2): track 0.00 -> 123.5 mm
- net /MUX_S2: track 20.1 -> 138.1 mm, vias 0 -> 3
- net GND: track 36.6 -> 149.6 mm, vias 12 -> 47
- net Net-(EX1-GPB2): track 0.00 -> 108.0 mm
- net /EXP2_INT: track 0.00 -> 103.9 mm, vias 0 -> 2
- net Net-(EX1-GPA3): track 0.00 -> 102.3 mm
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
Commit message: PCB V1.0 DONE
Parts:
- removed the C1 at (-79.1, -83.3)
- removed C54, C58: 100nF, Footprints:0603_C
- removed the C63 at (160.3, 42.4)
- removed the REF** at (-79.0, -91.5)
- removed the REF** at (-79.1, -95.2)
- removed the REF** at (-79.0, -86.5)
- removed the U2 at (-79.0, -86.5)
- added C52: 100nF, Footprints:0603_C, F.Cu at (205.6, 100.0)
- added R20: 330, Footprints:0603_R, F.Cu at (193.7, 90.8)
- added R21: 330, Footprints:0603_R, F.Cu at (193.7, 92.3)
- added R22: 330, Footprints:0603_R, F.Cu at (197.3, 112.0)
- added R23: 330, Footprints:0603_R, F.Cu at (195.8, 112.0)
- added R24: 330, Footprints:0603_R, F.Cu at (194.3, 112.0)
- J1: moved to B.Cu
- J4: value DIN 5 -> JST-EH; footprint Footprints:DIN_5 port -> Footprints:JST-EH port; moved to B.Cu
- R17, R18: value 330 -> 10k
- moved C71 237.0 mm to (278.0, 181.5)
- moved J2 144.8 mm to (146.9, 132.3), turned to 90 degrees
- moved C45 141.9 mm to (168.9, 141.2), turned to 90 degrees
- moved R17 140.5 mm to (164.5, 135.0), turned to 90 degrees
- moved FB1 139.8 mm to (166.7, 140.5)
- moved C73 139.0 mm to (170.4, 141.2), turned to 90 degrees
- moved Y1 135.7 mm to (166.9, 126.3), turned to 180 degrees
- moved C49 131.6 mm to (171.9, 141.2), turned to 90 degrees
- moved R14 130.1 mm to (183.0, 131.0), turned to -90 degrees
- moved C43 129.5 mm to (204.7, 148.9)
- moved C60 129.4 mm to (180.5, 131.0), turned to 90 degrees
- moved C80 126.6 mm to (165.7, 129.4), turned to 180 degrees
- moved C79 122.9 mm to (170.6, 125.5), turned to -90 degrees
- moved C50 118.3 mm to (171.7, 128.4), turned to 180 degrees
- moved C42 102.8 mm to (259.4, 102.5)
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- renumbered C52 to C51, C51 to C53, C53 to C63
Connections:
- net /SPI LED chain/SOFT_SPI_CLK renamed /SOFT_SPI_CLK
- net /SPI LED chain/SOFT_SPI_MOSI renamed /SOFT_SPI_MOSI
- DM3 pad 12: DISPLAY_RST -> D_IN_1
- EX2 pad 8: D_IN_1 -> DISPLAY_RST
- J1 pad A9: (no net) -> Net-(J1-VBUS)
- J1 pad B6: (no net) -> Net-(J1-D+)
- J1 pad B7: (no net) -> Net-(J1-D-)
- J3 pad 3: /SPI_MISO -> Net-(J3-MISO)
- J3 pad 4: /SPI_MOSI -> Net-(J3-MOSI)
- J3 pad 5: /SPI_SCK -> Net-(J3-SCK)
- R10 pad 1: Net-(U14-(PCINT19/OC2B/INT1)PD3) -> Net-(U14-(PCINT0/CLK0/ICP1)PB0)
- R11 pad 1: Net-(U14-(PCINT20/XCK/T0)PD4) -> Net-(U14-(PCINT1/OC1A)PB1)
- R17 pad 1: /RESET -> Net-(U14-(PCINT2/~{SS}/OC1B)PB2)
- R17 pad 2: /ATmega32u4/328p_RESET -> VCC
- R18 pad 2: Net-(J4-VCC) -> /DISPLAY_SS
- R19 pad 1: Net-(U15-(TXD1/INT3)PD3) -> /RESET
- R19 pad 2: Net-(J4-DATA) -> /ATmega32u4/328p_RESET
- U14 pad 1: Net-(U14-(PCINT19/OC2B/INT1)PD3) -> /DISPLAY_SS
- U14 pad 12: /MUX_S3 -> Net-(U14-(PCINT0/CLK0/ICP1)PB0)
- U14 pad 13: /DISPLAY_SS -> Net-(U14-(PCINT1/OC1A)PB1)
- U14 pad 14: unconnected-(U14-(PCINT2/~{SS}/OC1B)PB2-Pad14) -> Net-(U14-(PCINT2/~{SS}/OC1B)PB2)
- U14 pad 2: Net-(U14-(PCINT20/XCK/T0)PD4) -> /MUX_S3
- U15 pad 10: /SPI_MOSI -> Net-(J3-MOSI)
- U15 pad 11: /SPI_MISO -> Net-(J3-MISO)
- U15 pad 9: /SPI_SCK -> Net-(J3-SCK)
- U16 pad 1: Net-(J1-D+) -> Net-(J1-D-)
- U16 pad 3: Net-(J1-D-) -> Net-(J1-D+)
- U16 pad 4: Net-(R13-Pad1) -> Net-(R12-Pad1)
- U16 pad 6: Net-(R12-Pad1) -> Net-(R13-Pad1)
Routing:
- net VCC: track 884.2 -> 1782.1 mm, vias 0 -> 22
- net D_IN_1: track 150.4 -> 25.5 mm
- net /MUX_S3: track 22.4 -> 131.6 mm, vias 0 -> 4
- net /DISPLAY_SS: track 0.00 -> 105.8 mm, vias 0 -> 2
- net /SPI_MOSI: track 66.8 -> 164.1 mm, vias 2 -> 4
- net /SPI_SCK: track 69.0 -> 162.2 mm, vias 2 -> 4
- net /MUX_S0: track 68.8 -> 150.9 mm
- net /MUX_S1: track 67.9 -> 149.9 mm
- net /SOFT_SPI_MOSI: track 11.4 -> 90.7 mm
- net /SOFT_SPI_CLK: track 8.93 -> 88.2 mm
- net /ATmega32u4/328p_RESET: track 0.00 -> 57.6 mm
- net DISPLAY_RST: track 0.00 -> 44.5 mm, vias 0 -> 1
- net /RESET: track 0.00 -> 37.8 mm, vias 0 -> 3
- net /DMUX_OUT: track 0.00 -> 26.0 mm, vias 0 -> 2
- net Net-(J3-SCK): track 0.00 -> 22.0 mm
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- added copper zone on B.Cu, net GND
Other:
- board size 659.3 x 307 mm -> 287.4 x 138.4 mm

Commit message: last double-checks
Parts:
- moved C70 2.74 mm to (109.4, 147.6), turned to -90 degrees
- moved REF** 2.38 mm to (81.0, 154.8)
- moved C1 2.38 mm to (81.0, 146.0)
- moved C2 2.38 mm to (100.0, 146.1)
- moved C3 2.38 mm to (119.1, 146.2)
- moved C37 2.38 mm to (78.1, 154.8)
- moved C38 2.38 mm to (97.0, 154.8)
- moved C39 2.38 mm to (116.2, 154.8)
- moved C4 2.38 mm to (157.2, 146.0)
- moved C40 2.38 mm to (154.3, 154.8)
- moved C41 2.38 mm to (173.3, 154.8)
- moved C5 2.38 mm to (176.2, 146.0)
- moved D1 2.38 mm to (81.0, 149.7)
- moved D2 2.38 mm to (100.0, 149.7)
- moved D3 2.38 mm to (119.1, 149.7)
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- renumbered C64 to C13
Routing:
- net Net-(D5-SDO): track 141.5 -> 143.8 mm
- net Net-(D5-CKO): track 140.7 -> 143.1 mm
- net Net-(D2-CKO): track 12.8 -> 14.9 mm
- net Net-(AM1-I0): track 140.6 -> 139.1 mm
- net /SOFT_SPI_CLK: track 88.2 -> 86.8 mm
- net Net-(AM1-I12): track 128.0 -> 126.6 mm
- net /SOFT_SPI_MOSI: track 90.7 -> 89.3 mm
- net Net-(D2-SDO): track 12.8 -> 14.1 mm
- net Net-(AM1-I13): track 87.4 -> 86.1 mm
- net Net-(AM1-I14): track 65.6 -> 64.4 mm
- net Net-(AM1-I15): track 43.9 -> 42.8 mm
- net VCC: track 1782.1 -> 1783.0 mm
Other:
- board size 287.4 x 138.4 mm -> 287 x 138 mm
- board text added: "HARMORA 328 V1"
