File: PCB/Harmora.kicad_sch (KiCad schematic)
At the start: 23 parts, among them J5 128x64 2.42 inc, U14 ATmega328p-AU, Y1 16Mhz

Commit message: finished reworking pcb
Parts:
- removed J5: 128x64 2.42 inc, Footprints:SPI Screen PinHeader, symbol Symbols:SPI_OLED_Display
- removed R10, R11: 22, Footprints:0603_R, symbol Symbols:Resistor 0603
- removed R16, R17, R18: 10k, Footprints:0603_R, symbol Symbols:Resistor 0603
Connections:
- net SPI_SS: now reaches U14.14 ((PCINT2/~{SS}/OC1B)PB2)
- net 32U4_SS: no longer names the net of U14.23 ((ADC0/PCINT8)PC0)
- net DISPLAY_DR: no longer names the net of U14.30 ((RXD/PCINT16)PD0)
- net DISPLAY_SS: no longer names the net of U14.1 ((PCINT19/OC2B/INT1)PD3)
- no-connect marks 1 -> 6
Other:
- removed sheet SPI LED chain
- sheet ATmega32u4 ports: added 328P_SS; removed SPI_SS
- moved on the sheet: C13, C45, C49, C50, C60, C73, C79, C80, FB1, J2, R14, R19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
