File: PCB/schematic_pages/expanders.kicad_sch (KiCad schematic)
At the start: 32 parts

Commit message: pc is being
Parts:
- renumbered B16 to B14, B14 to B16
Connections:
- net D_IN_1: now also EX2.8 (GPB7); no longer EX1.22 (GPA1)
- net D_IN_21: now also EX2.7 (GPB6); no longer EX1.24 (GPA3)
- net D_IN_22: now also EX2.6 (GPB5); no longer EX1.23 (GPA2)
- net D_IN_23: now also EX2.5 (GPB4); no longer EX2.8 (GPB7)
- net at B16.1: now also EX1.6 (GPB5); no longer EX2.1 (GPB0)
- net at B6.1: now also EX1.23 (GPA2); no longer EX1.6 (GPB5)
- net at EX2.2 (GPB1): now also B23.1; no longer B15.1
- net at S1.2: now also EX2.1 (GPB0); no longer EX2.21 (GPA0)
- net at EX2.22 (GPA1): now also B18.1; no longer S2.2
- net at EX2.23 (GPA2): now also B4.1; no longer S3.2
- net at EX2.24 (GPA3): now also B7.1; no longer B21.1
- net at EX2.25 (GPA4): now also B19.1; no longer B22.1
- net at EX2.26 (GPA5): now also B20.1; no longer B23.1
- net at EX2.27 (GPA6): now also S2.2; no longer B7.1
- net at EX2.28 (GPA7): now also S3.2; no longer B4.1
- net at EX2.3 (GPB2): now also B22.1; no longer B14.1
- net at B17.1: now also EX2.21 (GPA0); no longer EX2.4 (GPB3)
- net at EX1.7 (GPB6): now also B15.1; no longer B9.1
- net at B10.1: now also EX1.27 (GPA6); no longer EX1.25 (GPA4)
- net at EX1.2 (GPB1): now also B8.1; no longer B2.1
- net at B11.1: now also EX1.25 (GPA4); no longer EX1.26 (GPA5)
- net at B12.1: now also EX1.28 (GPA7); no longer EX1.27 (GPA6)
- net at B13.1: now also EX1.26 (GPA5); no longer EX1.28 (GPA7)
- net at B3.1: now also EX1.24 (GPA3); no longer EX1.3 (GPB2)
- net at EX1.4 (GPB3): now also B2.1; no longer B8.1
- net at EX1.5 (GPB4): now also B9.1; no longer B5.1
- net at EX1.8 (GPB7): now also B14.1; no longer B24.1
- new net: B21.1, EX2.4 (GPB3)
- new net: B24.1, EX1.22 (GPA1)
- new net: B5.1, EX1.3 (GPB2)
Other:
- moved on the sheet: B14, B15, B16

Commit message: PCB V1.0 DONE
Connections:
- net D_IN_1 renamed DISPLAY_RST
Other:
- note removed: "ENCODER 4"
Changed lines of the file:
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@@
-		)
-	)
-	(text "ENCODER 4"
-		(exclude_from_sim no)
-		(at 112.014 122.174 0)
-		(effects
-			(font
-				(size 1.27 1.27)
-			)
-			(justify left)
 		)
 	)
@@
 			(width 0)
 			(type default)
-		)
-	)
-	(global_label "D_IN_1"
-		(shape input)
-		(at 102.87 121.92 0)
-		(fields_autoplaced yes)
-		(effects
-			(font
-				(size 1.27 1.27)
-				(color 221 133 0 1)
-			)
-			(justify left)
-		)
-		(property "Intersheetrefs" "${INTERSHEET_REFS}"
-			(at 112.2052 121.92 0)
-			(effects
-				(font
-					(size 1.27 1.27)
-				)
-				(justify left)
-				(hide yes)
-			)
 		)
 	)
@@
 			(effects
 				(font
+					(size 1.27 1.27)
+				)
+				(justify left)
+				(hide yes)
+			)
+		)
+	)
+	(global_label "DISPLAY_RST"
+		(shape input)
+		(at 102.87 121.92 0)
+		(fields_autoplaced yes)
+		(effects
+			(font
+				(size 1.27 1.27)
+				(color 221 133 0 1)
+			)
+			(justify left)
+		)
+		(property "Intersheetrefs" "${INTERSHEET_REFS}"
+			(at 117.8295 121.92 0)
+			(effects
+				(font

Commit message: finished reworking pcb
Connections:
- net DISPLAY_RST: no longer names the net of EX2.8 (GPB7)
- no-connect marks 3 -> 4
