File: PCB/schematic_pages/analog_mux.kicad_sch (KiCad schematic)
At the start: 33 parts, among them P1 10k, P2 10k, P3 10k, P4 10k, U1 SS49E, U10 SS49E, U11 SS49E, U12 SS49E, U2 SS49E, U3 SS49E, U4 SS49E, U5 SS49E, U6 SS49E, U7 SS49E, U8 SS49E, U9 SS49E

Commit message: pcb: piano done
Parts:
- renumbered P3 to P1, P4 to P2, P2 to P3, P1 to P4, R2 to R1, R3 to R2, R4 to R3, R5 to R4
Connections:
- net at U12.3 (OUTPUT): now also AM1.9 (I0); no longer AM1.20 (I11)
- net at U6.3 (OUTPUT): now also AM1.3 (I6); no longer AM1.4 (I5)
- net at U9.3 (OUTPUT): now also AM1.17 (I14); no longer AM1.23 (I8)
- net at AM1.16 (I15): now also U8.3 (OUTPUT); no longer R1.1
- net at R2.1: now also AM1.21 (I10); no longer AM1.17 (I14)
- net at AM1.18 (I13): now also U10.3 (OUTPUT); no longer R3.1
- net at AM1.19 (I12): now also U11.3 (OUTPUT); no longer R4.1
- net at AM1.2 (I7): now also U7.3 (OUTPUT); no longer U8.3 (OUTPUT)
- net at AM1.22 (I9): now also R3.1; no longer U10.3 (OUTPUT)
- net at U5.3 (OUTPUT): now also AM1.4 (I5); no longer AM1.5 (I4)
- net at U4.3 (OUTPUT): now also AM1.5 (I4); no longer AM1.6 (I3)
- net at U3.3 (OUTPUT): now also AM1.6 (I3); no longer AM1.7 (I2)
- net at U2.3 (OUTPUT): now also AM1.7 (I2); no longer AM1.8 (I1)
- net at U1.3 (OUTPUT): now also AM1.8 (I1); no longer AM1.9 (I0)
- new net: AM1.20 (I11), R1.1
- new net: AM1.23 (I8), R4.1
Changed lines of the file:
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@@
 		(on_board yes)
 		(dnp no)
-		(property "Reference" "R4"
+		(property "Reference" "R3"
 			(at 57.658 121.158 90)
 			(effects
@@
 			(project "pcb_schematics"
 				(path "/de43e009-b04c-42c1-b131-cdc664039a0d/333a86ff-2f60-4263-8580-754eb0fa7cf4"
-					(reference "R4")
+					(reference "R3")
 					(unit 1)
 				)
@@
 		(on_board yes)
 		(dnp no)
-		(property "Reference" "R2"
+		(property "Reference" "R1"
 			(at 57.658 126.238 90)
 			(effects
@@
 			(project "pcb_schematics"
 				(path "/de43e009-b04c-42c1-b131-cdc664039a0d/333a86ff-2f60-4263-8580-754eb0fa7cf4"
-					(reference "R2")
+					(reference "R1")
 					(unit 1)
 				)
@@
 		(dnp no)
 		(fields_autoplaced yes)
-		(property "Reference" "P4"
+		(property "Reference" "P2"
 			(at 104.14 140.97 90)
 			(effects
@@
 			(project "pcb_schematics"
 				(path "/de43e009-b04c-42c1-b131-cdc664039a0d/333a86ff-2f60-4263-8580-754eb0fa7cf4"
-					(reference "P4")
+					(reference "P2")
 					(unit 1)
 				)
@@
 		(dnp no)
 		(fields_autoplaced yes)
-		(property "Reference" "P1"
+		(property "Reference" "P4"
 			(at 62.23 140.97 90)
 			(effects
@@
 			(project "pcb_schematics"
 				(path "/de43e009-b04c-42c1-b131-cdc664039a0d/333a86ff-2f60-4263-8580-754eb0fa7cf4"
-					(reference "P1")
+					(reference "P4")
 					(unit 1)
 				)
@@
 		(dnp no)
 		(fields_autoplaced yes)
-		(property "Reference" "P2"
+		(property "Reference" "P3"
 			(at 76.2 140.97 90)
 			(effects
@@
 			(project "pcb_schematics"
 				(path "/de43e009-b04c-42c1-b131-cdc664039a0d/333a86ff-2f60-4263-8580-754eb0fa7cf4"
-					(reference "P2")
+					(reference "P3")
 					(unit 1)
 				)
@@
 		(on_board yes)
 		(dnp no)
-		(property "Reference" "R3"
+		(property "Reference" "R2"
 			(at 57.658 123.698 90)
 			(effects
@@
 			(project "pcb_schematics"
 				(path "/de43e009-b04c-42c1-b131-cdc664039a0d/333a86ff-2f60-4263-8580-754eb0fa7cf4"
-					(reference "R3")
+					(reference "R2")
 					(unit 1)
 				)
@@
 		(on_board yes)
 		(dnp no)
-		(property "Reference" "R5"
+		(property "Reference" "R4"
 			(at 57.658 118.618 90)
 			(effects
@@
 			(project "pcb_schematics"
 				(path "/de43e009-b04c-42c1-b131-cdc664039a0d/333a86ff-2f60-4263-8580-754eb0fa7cf4"
-					(reference "R5")
+					(reference "R4")
 					(unit 1)
 				)
@@
 		(dnp no)
 		(fields_autoplaced yes)
-		(property "Reference" "P3"
+		(property "Reference" "P1"
 			(at 90.17 140.97 90)
 			(effects
@@
 			(project "pcb_schematics"
 				(path "/de43e009-b04c-42c1-b131-cdc664039a0d/333a86ff-2f60-4263-8580-754eb0fa7cf4"
-					(reference "P3")
+					(reference "P1")
 					(unit 1)
 				)
