File: PCB/schematic_pages/digital_mux.kicad_sch (KiCad schematic)
At the start: 9 parts

Commit message: repo rearrange
Connections:
- net MUX2_OUT renamed DMUX_OUT
- net MUX_IN_0 renamed DMUX_S0
- net MUX_IN_1 renamed DMUX_S1
- net MUX_IN_2 renamed DMUX_S2
- net MUX_IN_3 renamed DMUX_S3

Commit message: new schematics
Parts:
- DM1: footprint (none) -> Footprints:74LVC1G157 SOT-363 2_1 MUX
- DM2, DM3: footprint (none) -> Footprints:74AC151SC SOIC-16 8_1 MUX
- EN1, EN2, EN3, EN4, EN5, EN6: footprint (none) -> Footprints:Rotary Encoder EC11E
Changed lines of the file:
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@@
 			)
 		)
-		(property "Footprint" ""
+		(property "Footprint" "Footprints:Rotary Encoder EC11E"
 			(at 199.39 62.23 0)
 			(effects
@@
 			)
 		)
-		(property "Footprint" ""
+		(property "Footprint" "Footprints:Rotary Encoder EC11E"
 			(at 138.43 62.23 0)
 			(effects
@@
 			)
 		)
-		(property "Footprint" ""
+		(property "Footprint" "Footprints:74AC151SC SOIC-16 8_1 MUX"
 			(at 93.98 83.82 0)
 			(effects
@@
 			)
 		)
-		(property "Footprint" ""
+		(property "Footprint" "Footprints:Rotary Encoder EC11E"
 			(at 158.75 62.23 0)
 			(effects
@@
 			)
 		)
-		(property "Footprint" ""
+		(property "Footprint" "Footprints:Rotary Encoder EC11E"
 			(at 179.07 62.23 0)
 			(effects
@@
 			)
 		)
-		(property "Footprint" ""
+		(property "Footprint" "Footprints:74LVC1G157 SOT-363 2_1 MUX"
 			(at 63.5 106.68 0)
 			(effects
@@
 			)
 		)
-		(property "Footprint" ""
+		(property "Footprint" "Footprints:Rotary Encoder EC11E"
 			(at 118.11 62.23 0)
 			(effects
@@
 			)
 		)
-		(property "Footprint" ""
+		(property "Footprint" "Footprints:Rotary Encoder EC11E"
 			(at 219.71 62.23 0)
 			(effects
@@
 			)
 		)
-		(property "Footprint" ""
+		(property "Footprint" "Footprints:74AC151SC SOIC-16 8_1 MUX"
 			(at 93.98 120.65 0)
 			(effects

Commit message: ISP ports, RESET lines, MIDI DIN 5
Connections:
- net DISPLAY_RST: now reaches DM3.13 (I6)
- no-connect marks 4 -> 3
Changed lines of the file:
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@@
 		(at 102.87 132.08)
 	)
-	(no_connect
-		(at 102.87 129.54)
-	)
 	(wire
 		(pts
@@
 		)
 	)
+	(global_label "DISPLAY_RST"
+		(shape input)
+		(at 102.87 129.54 0)
+		(fields_autoplaced yes)
+		(effects
+			(font
+				(size 1.27 1.27)
+			)
+			(justify left)
+		)
+		(property "Intersheetrefs" "${INTERSHEET_REFS}"
+			(at 117.8295 129.54 0)
+			(effects
+				(font
+					(size 1.27 1.27)
+				)
+				(justify left)
+				(hide yes)
+			)
+		)
+	)

Commit message: longahh day
Connections:
- net DISPLAY_RST: now also DM3.12 (I7); no longer DM3.13 (I6)
- net at EN5.1 (A): now also DM3.1 (I3); no longer DM3.4 (I0)
- net at EN5.3 (B): now also DM3.2 (I2); no longer DM3.3 (I1)
- net at EN5.4 (SW): now also DM3.14 (I5); no longer DM3.15 (I4)
- net at EN2.1 (A): now also DM2.3 (I1); no longer DM2.2 (I2)
- net at EN2.3 (B): now also DM2.4 (I0); no longer DM2.1 (I3)
- net at DM2.12 (I7): now also EN4.1 (A); no longer EN4.3 (B)
- net at DM2.13 (I6): now also EN4.3 (B); no longer EN4.1 (A)
- net at DM2.14 (I5): now also EN3.1 (A); no longer EN3.3 (B)
- net at DM2.15 (I4): now also EN3.3 (B); no longer EN3.1 (A)
- net at EN1.3 (B): now also DM2.2 (I2); no longer DM2.3 (I1)
- net at EN1.1 (A): now also DM2.1 (I3); no longer DM2.4 (I0)
- net at EN6.1 (A): now also DM3.3 (I1); no longer DM3.2 (I2)
- net at EN6.3 (B): now also DM3.4 (I0); no longer DM3.1 (I3)
- net at EN6.4 (SW): now also DM3.15 (I4); no longer DM3.14 (I5)

Commit message: pc is being
Connections:
- net at EN5.1 (A): now also DM3.2 (I2); no longer DM3.1 (I3)
- net at EN5.3 (B): now also DM3.1 (I3); no longer DM3.2 (I2)
- net at EN5.4 (SW): now also DM3.3 (I1); no longer DM3.14 (I5)
- net at DM2.12 (I7): now also EN4.3 (B); no longer EN4.1 (A)
- net at DM2.13 (I6): now also EN4.1 (A); no longer EN4.3 (B)
- net at EN6.1 (A): now also DM3.15 (I4); no longer DM3.3 (I1)
- net at EN6.3 (B): now also DM3.14 (I5); no longer DM3.4 (I0)
- net at EN6.4 (SW): now also DM3.4 (I0); no longer DM3.15 (I4)
Changed lines of the file:
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@@
 	(wire
 		(pts
-			(xy 208.28 127) (xy 102.87 127)
-		)
-		(stroke
-			(width 0)
-			(type default)
-		)
-	)
-	(wire
-		(pts
-			(xy 201.93 71.12) (xy 201.93 116.84)
-		)
-		(stroke
-			(width 0)
-			(type default)
-		)
-	)
-	(wire
-		(pts
-			(xy 176.53 92.71) (xy 176.53 71.12)
+			(xy 217.17 127) (xy 102.87 127)
+		)
+		(stroke
+			(width 0)
+			(type default)
+		)
+	)
+	(wire
+		(pts
+			(xy 201.93 71.12) (xy 201.93 114.3)
+		)
+		(stroke
+			(width 0)
+			(type default)
+		)
+	)
+	(wire
+		(pts
+			(xy 217.17 71.12) (xy 217.17 127)
 		)
 		(stroke
@@
 	(wire
 		(pts
-			(xy 102.87 121.92) (xy 222.25 121.92)
-		)
-		(stroke
-			(width 0)
-			(type default)
-		)
-	)
-	(wire
-		(pts
-			(xy 217.17 119.38) (xy 102.87 119.38)
+			(xy 102.87 92.71) (xy 181.61 92.71)
+		)
+		(stroke
+			(width 0)
+			(type default)
+		)
+	)
+	(wire
+		(pts
+			(xy 187.96 119.38) (xy 102.87 119.38)
+		)
+		(stroke
+			(width 0)
+			(type default)
+		)
+	)
+	(wire
+		(pts
+			(xy 102.87 124.46) (xy 222.25 124.46)
+		)
+		(stroke
+			(width 0)
+			(type default)
+		)
+	)
+	(wire
+		(pts
+			(xy 196.85 116.84) (xy 102.87 116.84)
+		)
+		(stroke
+			(width 0)
+			(type default)
+		)
+	)
+	(wire
+		(pts
+			(xy 187.96 53.34) (xy 187.96 119.38)
 		)
 		(stroke
@@
 	(wire
 		(pts
-			(xy 222.25 121.92) (xy 222.25 71.12)
-		)
-		(stroke
-			(width 0)
-			(type default)
-		)
-	)
-	(wire
-		(pts
 			(xy 156.21 87.63) (xy 156.21 71.12)
 		)
@@
 	(wire
 		(pts
-			(xy 102.87 95.25) (xy 181.61 95.25)
-		)
-		(stroke
-			(width 0)
-			(type default)
-		)
-	)
-	(wire
-		(pts
 			(xy 196.85 53.34) (xy 187.96 53.34)
 		)
@@
 	(wire
 		(pts
-			(xy 217.17 71.12) (xy 217.17 119.38)
-		)
-		(stroke
-			(width 0)
-			(type default)
-		)
-	)
-	(wire
-		(pts
 			(xy 161.29 90.17) (xy 161.29 71.12)
 		)
@@
 	(wire
 		(pts
-			(xy 102.87 92.71) (xy 176.53 92.71)
-		)
-		(stroke
-			(width 0)
-			(type default)
-		)
-	)
-	(wire
-		(pts
-			(xy 196.85 114.3) (xy 196.85 71.12)
+			(xy 176.53 95.25) (xy 102.87 95.25)
+		)
+		(stroke
+			(width 0)
+			(type default)
+		)
+	)
+	(wire
+		(pts
+			(xy 222.25 71.12) (xy 222.25 124.46)
 		)
 		(stroke
@@
 	(wire
 		(pts
-			(xy 208.28 53.34) (xy 208.28 127)
-		)
-		(stroke
-			(width 0)
-			(type default)
-		)
-	)
-	(wire
-		(pts
 			(xy 72.39 129.54) (xy 85.09 129.54)
 		)
@@
 	(wire
 		(pts
+			(xy 208.28 53.34) (xy 208.28 121.92)
+		)
+		(stroke
+			(width 0)
+			(type default)
+		)
+	)
+	(wire
+		(pts
+			(xy 176.53 71.12) (xy 176.53 95.25)
+		)
+		(stroke
+			(width 0)
+			(type default)
+		)
+	)
+	(wire
+		(pts
+			(xy 196.85 71.12) (xy 196.85 116.84)
+		)
+		(stroke
+			(width 0)
+			(type default)
+		)
+	)
+	(wire
+		(pts
 			(xy 82.55 100.33) (xy 93.98 100.33)
 		)
@@
 	(wire
 		(pts
-			(xy 201.93 116.84) (xy 102.87 116.84)
-		)
-		(stroke
-			(width 0)
-			(type default)
-		)
-	)
-	(wire
-		(pts
-			(xy 187.96 124.46) (xy 102.87 124.46)
-		)
-		(stroke
-			(width 0)
-			(type default)
-		)
-	)
-	(wire
-		(pts
 			(xy 85.09 124.46) (xy 81.28 124.46)
 		)
@@
 	(wire
 		(pts
-			(xy 102.87 114.3) (xy 196.85 114.3)
-		)
-		(stroke
-			(width 0)
-			(type default)
-		)
-	)
-	(wire
-		(pts
-			(xy 187.96 53.34) (xy 187.96 124.46)
+			(xy 102.87 114.3) (xy 201.93 114.3)
 		)
 		(stroke
@@
 	(wire
 		(pts
-			(xy 181.61 95.25) (xy 181.61 71.12)
-		)
-		(stroke
+			(xy 208.28 121.92) (xy 102.87 121.92)
+		)
+		(stroke
+			(width 0)
+			(type default)
+		)
+	)
+	(wire
+		(pts
+			(xy 181.61 71.12) (xy 181.61 92.71)
+		)
+		(stroke

Commit message: PCB V1.0 DONE
Connections:
- net DISPLAY_RST is gone; now on net D_IN_1: DM3.12 (I7)
Other:
- note added: "ENCODER 4"
Changed lines of the file:
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@@
 	(generator_version "9.0")
 	(paper "A4")
+	(text "ENCODER 4"
+		(exclude_from_sim no)
+		(at 112.014 129.794 0)
+		(effects
+			(font
+				(size 1.27 1.27)
+			)
+			(justify left)
+		)
+	)
 	(junction
 		(at 93.98 137.16)
@@
 			(width 0)
 			(type default)
-		)
-	)
-	(global_label "DISPLAY_RST"
-		(shape input)
-		(at 102.87 129.54 0)
-		(fields_autoplaced yes)
-		(effects
-			(font
-				(size 1.27 1.27)
-			)
-			(justify left)
-		)
-		(property "Intersheetrefs" "${INTERSHEET_REFS}"
-			(at 117.8295 129.54 0)
-			(effects
-				(font
-					(size 1.27 1.27)
-				)
-				(justify left)
-				(hide yes)
-			)
 		)
 	)
@@
 			(effects
 				(font
+					(size 1.27 1.27)
+				)
+				(justify left)
+				(hide yes)
+			)
+		)
+	)
+	(global_label "D_IN_1"
+		(shape input)
+		(at 102.87 129.54 0)
+		(fields_autoplaced yes)
+		(effects
+			(font
+				(size 1.27 1.27)
+				(color 221 133 0 1)
+			)
+			(justify left)
+		)
+		(property "Intersheetrefs" "${INTERSHEET_REFS}"
+			(at 112.2052 129.54 0)
+			(effects
+				(font

Commit message: finished reworking pcb
Parts:
- added R17, R26, R27, R28, R29, R30, R31, R32, R33, R34, R35, R36: 10k, Footprints:0603_R, symbol Symbols:Resistor 0603
Connections:
- net VCC: now also DM2.16 (VCC), DM3.16 (VCC), R17.2, R26.2, R27.2, R28.2, R29.2, R30.2, R31.2, R32.2, R33.2, R34.2, R35.2, R36.2; no longer DM2. (VCC), DM3. (VCC)
- net at DM3.2 (I2), EN5.1 (A): now also R28.1
- net at DM3.1 (I3), EN5.3 (B): now also R27.1
- net at DM2.3 (I1), EN2.1 (A): now also R34.1
- net at DM2.4 (I0), EN2.3 (B): now also R33.1
- net at DM2.1 (I3), EN1.1 (A): now also R36.1
- net at DM2.12 (I7), EN4.3 (B): now also R29.1
- net at DM2.13 (I6), EN4.1 (A): now also R30.1
- net at DM2.14 (I5), EN3.1 (A): now also R32.1
- net at DM2.15 (I4), EN3.3 (B): now also R31.1
- net at DM2.2 (I2), EN1.3 (B): now also R35.1
- net at DM3.15 (I4), EN6.1 (A): now also R26.1
- net at DM3.14 (I5), EN6.3 (B): now also R17.1
Other:
- moved on the sheet: DM1, EN1, EN2, EN3, EN4, EN5, EN6
