File: PCB/schematic_pages/schematic_pages/SPI_LED_chain.kicad_sch (KiCad schematic)
At the start: 55 parts

Commit message: finished reworking pcb
Parts:
- renumbered C5 to C1, C1 to C10, C9 to C11, C15 to C12, C3 to C14, C11 to C15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
Other:
- moved on the sheet: C1, C10, C11, C12, C14, C15, C16, C17, C18, C19, C2, C20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
